File: SplitKeyboard/SplitKeyboard.kicad_pcb (KiCad board)
At the start: 2 copper layers, 3.6 x 3.1 mm, 238 parts, among them J1 LED, P2 OLED, SW0 SW_Push, SW1 SW_Push, SW10 SW_DownArrow, SW13 SW_RightArrow, SW14 SW_Push, SW15 SW_Push, SW16 Rotary_Encoder_Switch, SW2 SW_Push, SW3 SW_Push, SW4 SW_Push, SW5 SW_Push, SW6 SW_Push, SW7 SW_Push, SW8 SW_Push, SW9 SW_Push, U1 ARDUINO_MICRO_SHIELD

Commit message: minivan with RGB knob and led display
Parts:
- added REF**: Stabilizer_Cherry_MX_2u, Mech5:Stabilizer_Cherry_MX_2u, F.Cu at (355.5, 139.1)
- added REF**: Stabilizer_Cherry_MX_2u, Mech5:Stabilizer_Cherry_MX_2u, F.Cu at (348.4, 110.5)
- added REF**: Stabilizer_Cherry_MX_2u, Mech5:Stabilizer_Cherry_MX_2u, F.Cu at (341.2, 167.7)
- added REF**: Stabilizer_Cherry_MX_2u, Mech5:Stabilizer_Cherry_MX_2u, F.Cu at (68.0, 147.6)
- added REF**: Stabilizer_Cherry_MX_2u, Mech5:Stabilizer_Cherry_MX_2u, F.Cu at (65.6, 128.5)
- added REF**: Stabilizer_Cherry_MX_2u, Mech5:Stabilizer_Cherry_MX_2u, F.Cu at (179.9, 185.7)
- added Ref**: Val**, Mech1:M2_HOLE_v3, F.Cu at (108.7, 110.9)
- added Ref**: Val**, Mech1:M2_HOLE_v3, F.Cu at (250.0, 92.1)
- added Ref**: Val**, Mech1:M2_HOLE_v3, F.Cu at (385.0, 101.6)
- added Ref**: Val**, Mech1:M2_HOLE_v3, F.Cu at (331.0, 109.5)
- added Ref**: Val**, Mech1:M2_HOLE_v3, F.Cu at (385.0, 193.7)
- added Ref**: Val**, Mech1:M2_HOLE_v3, F.Cu at (319.9, 162.7)
- added Ref**: Val**, Mech1:M2_HOLE_v3, F.Cu at (122.2, 185.7)
- added Ref**: Val**, Mech1:M2_HOLE_v3, F.Cu at (190.5, 166.7)
- added Ref**: Val**, Mech1:M2_HOLE_v3, F.Cu at (192.1, 72.2)
- added Ref**: Val**, Mech1:M2_HOLE_v3, F.Cu at (39.7, 70.6)
- added Ref**: Val**, Mech1:M2_HOLE_v3, F.Cu at (37.3, 188.1)
- added Ref**: Val**, Mech1:M2_HOLE_v3, F.Cu at (261.9, 131.0)
- added Ref**: Val**, Mech1:M2_HOLE_v3, F.Cu at (234.2, 188.9)
- added Ref**: Val**, Mech1:M2_HOLE_v3, F.Cu at (218.3, 148.4)
- moved D4 331.7 mm to (58.8, 158.2)
- moved D76 331.3 mm to (48.9, 143.6)
- moved D75 331.3 mm to (165.1, 183.1)
- moved D9 330.5 mm to (81.5, 158.4)
- moved D23 330.5 mm to (148.2, 138.0)
- moved D30 330.5 mm to (172.0, 99.9)
- moved D32 330.5 mm to (186.3, 138.0)
- moved D74 330.5 mm to (172.0, 74.5)
- moved JTRRS3 330.5 mm to (132.3, 56.3)
- moved JTRRS5 330.5 mm to (164.1, 56.3)
- moved JTRRS6 330.5 mm to (148.2, 56.3)
- moved LED29 330.5 mm to (179.9, 191.2)
- moved LED37 330.5 mm to (132.3, 153.1)
- moved LED44 330.5 mm to (156.1, 89.6)
- moved SW5 330.5 mm to (156.1, 109.5)
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Connections:
- D33 pad 1: Fila4 -> (no net)
- D33 pad 2: Net-(D33-Pad2) -> (no net)
- D34 pad 1: Fila1 -> (no net)
- D34 pad 2: Net-(D34-Pad2) -> (no net)
- D35 pad 1: Fila6 -> (no net)
- D35 pad 2: Net-(D35-Pad2) -> (no net)
- D36 pad 1: Fila3 -> (no net)
- D36 pad 2: Net-(D36-Pad2) -> (no net)
- D37 pad 1: Fila4 -> (no net)
- D37 pad 2: Net-(D37-Pad2) -> (no net)
- D38 pad 1: Fila1 -> (no net)
- D38 pad 2: Net-(D38-Pad2) -> (no net)
- D39 pad 1: Fila6 -> (no net)
- D39 pad 2: Net-(D39-Pad2) -> (no net)
- D40 pad 1: Fila3 -> (no net)
- D40 pad 2: Net-(D40-Pad2) -> (no net)
- D41 pad 1: Fila4 -> (no net)
- D41 pad 2: Net-(D41-Pad2) -> (no net)
- D42 pad 1: Fila1 -> (no net)
- D42 pad 2: Net-(D42-Pad2) -> (no net)
- D43 pad 1: Fila6 -> (no net)
- D43 pad 2: Net-(D43-Pad2) -> (no net)
- D44 pad 1: Fila3 -> (no net)
- D44 pad 2: Net-(D44-Pad2) -> (no net)
- D45 pad 1: Fila4 -> (no net)
- D45 pad 2: Net-(D45-Pad2) -> (no net)
- D46 pad 1: Fila1 -> (no net)
- D46 pad 2: Net-(D46-Pad2) -> (no net)
- D47 pad 1: Fila6 -> (no net)
- D47 pad 2: Net-(D47-Pad2) -> (no net)
- D48 pad 1: Fila3 -> (no net)
- D48 pad 2: Net-(D48-Pad2) -> (no net)
- D49 pad 1: Fila4 -> (no net)
- D49 pad 2: Net-(D49-Pad2) -> (no net)
- D50 pad 1: Fila5 -> (no net)
- D50 pad 2: Net-(D50-Pad2) -> (no net)
- D51 pad 1: Fila1 -> (no net)
- D51 pad 2: Net-(D51-Pad2) -> (no net)
- D52 pad 1: Fila6 -> (no net)
- D52 pad 2: Net-(D52-Pad2) -> (no net)
- D53 pad 1: Fila3 -> (no net)
- D53 pad 2: Net-(D53-Pad2) -> (no net)
- D54 pad 1: Fila1 -> (no net)
- D54 pad 2: Net-(D54-Pad2) -> (no net)
- D55 pad 1: Fila6 -> (no net)
- D55 pad 2: Net-(D55-Pad2) -> (no net)
- D56 pad 1: Fila3 -> (no net)
- D56 pad 2: Net-(D56-Pad2) -> (no net)
- D57 pad 1: Fila4 -> (no net)
- D57 pad 2: Net-(D57-Pad2) -> (no net)
- D58 pad 1: Fila5 -> (no net)
- D58 pad 2: Net-(D58-Pad2) -> (no net)
- D59 pad 1: Fila1 -> (no net)
- D59 pad 2: Net-(D59-Pad2) -> (no net)
- D60 pad 1: Fila6 -> (no net)
- D60 pad 2: Net-(D60-Pad2) -> (no net)
- D61 pad 1: Fila5 -> (no net)
- D61 pad 2: Net-(D61-Pad2) -> (no net)
- D62 pad 1: Fila1 -> (no net)
- D62 pad 2: Net-(D62-Pad2) -> (no net)
- D63 pad 1: Fila6 -> (no net)
- D63 pad 2: Net-(D63-Pad2) -> (no net)
- D64 pad 1: Fila5 -> (no net)
- D64 pad 2: Net-(D64-Pad2) -> (no net)
- D65 pad 1: Fila5 -> (no net)
- D65 pad 2: Net-(D65-Pad2) -> (no net)
- D66 pad 1: Fila3 -> (no net)
- D66 pad 2: Net-(D66-Pad2) -> (no net)
- D67 pad 1: Fila4 -> (no net)
- D67 pad 2: Net-(D67-Pad2) -> (no net)
- D68 pad 1: Fila5 -> (no net)
- D68 pad 2: Net-(D68-Pad2) -> (no net)
- JTRRS1 pad 1: Columna7 -> (no net)
- JTRRS1 pad 2: Columna6 -> (no net)
- JTRRS1 pad 3: Columna5 -> (no net)
- JTRRS1 pad 4: Columna8 -> (no net)
- JTRRS2 pad 1: Columna2 -> (no net)
- JTRRS2 pad 2: Columna3 -> (no net)
- JTRRS2 pad 3: Columna4 -> (no net)
- JTRRS2 pad 4: Columna16 -> (no net)
- JTRRS7 pad 1: Fila6 -> (no net)
- JTRRS7 pad 2: Fila3 -> (no net)
- JTRRS7 pad 3: Fila4 -> (no net)
- JTRRS7 pad 4: Fila1 -> (no net)
- JTRRS8 pad 1: GND -> (no net)
- JTRRS8 pad 2: LEDTRRS -> (no net)
- JTRRS8 pad 3: VCC -> (no net)
- JTRRS8 pad 4: Fila5 -> (no net)
- LED10 pad 1: VCC -> (no net)
- LED10 pad 2: Net-(LED10-Pad2) -> (no net)
- LED10 pad 3: GND -> (no net)
- LED10 pad 4: Net-(LED10-Pad4) -> (no net)
- LED13 pad 1: VCC -> (no net)
- LED13 pad 2: Net-(LED13-Pad2) -> (no net)
- LED13 pad 3: GND -> (no net)
- LED13 pad 4: Net-(LED13-Pad4) -> (no net)
- LED14 pad 1: VCC -> (no net)
- LED14 pad 2: Net-(LED14-Pad2) -> (no net)
- LED14 pad 3: GND -> (no net)
- LED14 pad 4: Net-(LED14-Pad4) -> (no net)
- LED17 pad 1: VCC -> (no net)
- LED17 pad 2: Net-(LED10-Pad4) -> (no net)
- LED17 pad 3: GND -> (no net)
- LED17 pad 4: Net-(LED17-Pad4) -> (no net)
- LED20 pad 1: VCC -> (no net)
- LED20 pad 2: Net-(LED20-Pad2) -> (no net)
- LED20 pad 3: GND -> (no net)
- LED20 pad 4: Net-(LED13-Pad2) -> (no net)
- LED21 pad 1: VCC -> (no net)
- LED21 pad 2: Net-(LED21-Pad2) -> (no net)
- LED21 pad 3: GND -> (no net)
- LED21 pad 4: Net-(LED14-Pad2) -> (no net)
- LED24 pad 1: VCC -> (no net)
- LED24 pad 2: Net-(LED17-Pad4) -> (no net)
- LED24 pad 3: GND -> (no net)
- LED24 pad 4: Net-(LED24-Pad4) -> (no net)
- LED27 pad 1: VCC -> (no net)
- LED27 pad 2: Net-(LED27-Pad2) -> (no net)
- LED27 pad 3: GND -> (no net)
- LED27 pad 4: Net-(LED20-Pad2) -> (no net)
- LED28 pad 1: VCC -> (no net)
- LED28 pad 2: Net-(LED28-Pad2) -> (no net)
- LED28 pad 3: GND -> (no net)
- LED28 pad 4: Net-(LED21-Pad2) -> (no net)
- LED33 pad 1: VCC -> (no net)
- LED33 pad 2: Net-(LED33-Pad2) -> (no net)
- LED33 pad 3: GND -> (no net)
- LED33 pad 4: Net-(LED27-Pad2) -> (no net)
- LED34 pad 1: VCC -> (no net)
- LED34 pad 2: Net-(LED24-Pad4) -> (no net)
- LED34 pad 3: GND -> (no net)
- LED34 pad 4: Net-(LED34-Pad4) -> (no net)
- LED35 pad 1: VCC -> (no net)
- LED35 pad 2: Net-(LED35-Pad2) -> (no net)
- LED35 pad 3: GND -> (no net)
- LED35 pad 4: Net-(LED28-Pad2) -> (no net)
- LED4 pad 1: VCC -> (no net)
- LED4 pad 2: Net-(LED4-Pad2) -> (no net)
- LED4 pad 3: GND -> (no net)
- LED4 pad 4: LEDTRRS -> (no net)
- LED40 pad 1: VCC -> (no net)
- LED40 pad 2: Net-(LED40-Pad2) -> (no net)
- LED40 pad 3: GND -> (no net)
- LED40 pad 4: Net-(LED33-Pad2) -> (no net)
- LED41 pad 1: VCC -> (no net)
- LED41 pad 2: Net-(LED34-Pad4) -> (no net)
- LED41 pad 3: GND -> (no net)
- LED41 pad 4: Net-(LED41-Pad4) -> (no net)
- LED42 pad 1: VCC -> (no net)
- LED42 pad 2: Net-(LED42-Pad2) -> (no net)
- LED42 pad 3: GND -> (no net)
- LED42 pad 4: Net-(LED35-Pad2) -> (no net)
- LED45 pad 1: VCC -> (no net)
- LED45 pad 2: Net-(LED41-Pad4) -> (no net)
- LED45 pad 3: GND -> (no net)
- LED45 pad 4: Net-(LED45-Pad4) -> (no net)
- LED48 pad 1: VCC -> (no net)
- LED48 pad 2: Net-(LED48-Pad2) -> (no net)
- LED48 pad 3: GND -> (no net)
- LED48 pad 4: Net-(LED40-Pad2) -> (no net)
- LED49 pad 1: VCC -> (no net)
- LED49 pad 2: Net-(LED49-Pad2) -> (no net)
- LED49 pad 3: GND -> (no net)
- LED49 pad 4: Net-(LED42-Pad2) -> (no net)
- LED5 pad 1: VCC -> (no net)
- LED5 pad 2: Net-(LED13-Pad4) -> (no net)
- LED5 pad 3: GND -> (no net)
- LED5 pad 4: Net-(LED4-Pad2) -> (no net)
- LED52 pad 1: VCC -> (no net)
- LED52 pad 2: Net-(LED45-Pad4) -> (no net)
- LED52 pad 3: GND -> (no net)
- LED52 pad 4: Net-(LED52-Pad4) -> (no net)
- LED55 pad 1: VCC -> (no net)
- LED55 pad 2: Net-(LED55-Pad2) -> (no net)
- LED55 pad 3: GND -> (no net)
- LED55 pad 4: Net-(LED48-Pad2) -> (no net)
- LED56 pad 1: VCC -> (no net)
- LED56 pad 2: Net-(LED56-Pad2) -> (no net)
- LED56 pad 3: GND -> (no net)
- LED56 pad 4: Net-(LED49-Pad2) -> (no net)
- LED59 pad 1: VCC -> (no net)
- LED59 pad 2: Net-(LED52-Pad4) -> (no net)
- LED59 pad 3: GND -> (no net)
- LED59 pad 4: Net-(LED59-Pad4) -> (no net)
- LED6 pad 1: VCC -> (no net)
- LED6 pad 2: Net-(LED6-Pad2) -> (no net)
- LED6 pad 3: GND -> (no net)
- LED6 pad 4: Net-(LED10-Pad2) -> (no net)
- LED62 pad 1: VCC -> (no net)
- LED62 pad 2: Net-(LED62-Pad2) -> (no net)
- LED62 pad 3: GND -> (no net)
- LED62 pad 4: Net-(LED55-Pad2) -> (no net)
- LED67 pad 1: VCC -> (no net)
- LED67 pad 2: Net-(LED67-Pad2) -> (no net)
- LED67 pad 3: GND -> (no net)
- LED67 pad 4: Net-(LED62-Pad2) -> (no net)
- LED68 pad 1: VCC -> (no net)
- LED68 pad 2: Net-(LED59-Pad4) -> (no net)
- LED68 pad 3: GND -> (no net)
- LED68 pad 4: Net-(LED67-Pad2) -> (no net)
- LED69 pad 1: VCC -> (no net)
- LED69 pad 2: Net-(LED69-Pad2) -> (no net)
- LED69 pad 3: GND -> (no net)
- LED69 pad 4: Net-(LED69-Pad4) -> (no net)
- LED7 pad 1: VCC -> (no net)
- LED7 pad 2: Net-(LED14-Pad4) -> (no net)
- LED7 pad 3: GND -> (no net)
- LED7 pad 4: Net-(LED6-Pad2) -> (no net)
- LED70 pad 1: VCC -> (no net)
- LED70 pad 2: Net-(LED70-Pad2) -> (no net)
- LED70 pad 3: GND -> (no net)
- LED70 pad 4: Net-(LED69-Pad2) -> (no net)
- LED71 pad 1: VCC -> (no net)
- LED71 pad 2: Net-(LED71-Pad2) -> (no net)
- LED71 pad 3: GND -> (no net)
- LED71 pad 4: Net-(LED70-Pad2) -> (no net)
- LED72 pad 1: VCC -> (no net)
- LED72 pad 2: Net-(LED72-Pad2) -> (no net)
- LED72 pad 3: GND -> (no net)
- LED72 pad 4: Net-(LED56-Pad2) -> (no net)
- LED73 pad 1: VCC -> (no net)
- LED73 pad 2: Net-(LED73-Pad2) -> (no net)
- LED73 pad 3: GND -> (no net)
- LED73 pad 4: Net-(LED71-Pad2) -> (no net)
- LED74 pad 1: VCC -> (no net)
- LED74 pad 2: Net-(LED69-Pad4) -> (no net)
- LED74 pad 3: GND -> (no net)
- LED74 pad 4: Net-(LED72-Pad2) -> (no net)
- LED75 pad 1: VCC -> (no net)
- LED75 pad 2: Net-(LED75-Pad2) -> (no net)
- LED75 pad 3: GND -> (no net)
- LED75 pad 4: Net-(LED73-Pad2) -> (no net)
- SW+1 pad 1: Net-(D55-Pad2) -> (no net)
- SW+1 pad 2: Columna3 -> (no net)
- SW0 pad 1: Net-(D46-Pad2) -> (no net)
- SW0 pad 2: Columna5 -> (no net)
- SW10 pad 1: Net-(D61-Pad2) -> (no net)
- SW10 pad 2: Columna3 -> (no net)
- SW13 pad 1: Net-(D68-Pad2) -> (no net)
- SW13 pad 2: Columna2 -> (no net)
- SW14 pad 1: Net-(D48-Pad2) -> (no net)
- SW14 pad 2: Columna5 -> (no net)
- SW15 pad 1: Net-(D52-Pad2) -> (no net)
- SW15 pad 2: Columna4 -> (no net)
- SW7 pad 1: Net-(D34-Pad2) -> (no net)
- SW7 pad 2: Columna8 -> (no net)
- SW8 pad 1: Net-(D38-Pad2) -> (no net)
- SW8 pad 2: Columna7 -> (no net)
- SW9 pad 1: Net-(D42-Pad2) -> (no net)
- SW9 pad 2: Columna6 -> (no net)
- SWCtrlright1 pad 1: Net-(D58-Pad2) -> (no net)
- SWCtrlright1 pad 2: Columna6 -> (no net)
- SWLeftArrow1 pad 1: Net-(D64-Pad2) -> (no net)
- SWLeftArrow1 pad 2: Columna4 -> (no net)
- SWUpArrow1 pad 1: Net-(D65-Pad2) -> (no net)
- SWUpArrow1 pad 2: Columna5 -> (no net)
- SWaltgr1 pad 1: Net-(D50-Pad2) -> (no net)
- SWaltgr1 pad 2: Columna7 -> (no net)
- SWbackslash1 pad 1: Net-(D59-Pad2) -> (no net)
- SWbackslash1 pad 2: Columna2 -> (no net)
- SWcomilla1 pad 1: Net-(D51-Pad2) -> (no net)
- SWcomilla1 pad 2: Columna4 -> (no net)
- SWcomma1 pad 1: Net-(D41-Pad2) -> (no net)
- SWcomma1 pad 2: Columna6 -> (no net)
- SWend1 pad 1: Net-(D63-Pad2) -> (no net)
- SWend1 pad 2: Columna16 -> (no net)
- SWenter1 pad 1: Net-(D60-Pad2) -> (no net)
- SWenter1 pad 2: Columna2 -> (no net)
- SWguion1 pad 1: Net-(D49-Pad2) -> (no net)
- SWguion1 pad 2: Columna4 -> (no net)
- SWhome1 pad 1: Net-(D62-Pad2) -> (no net)
- SWhome1 pad 2: Columna16 -> (no net)
- SWi1 pad 1: Net-(D39-Pad2) -> (no net)
- SWi1 pad 2: Columna7 -> (no net)
- SWj1 pad 1: Net-(D36-Pad2) -> (no net)
- SWj1 pad 2: Columna8 -> (no net)
- SWk1 pad 1: Net-(D40-Pad2) -> (no net)
- SWk1 pad 2: Columna7 -> (no net)
- SWl1 pad 1: Net-(D44-Pad2) -> (no net)
- SWl1 pad 2: Columna6 -> (no net)
- SWm1 pad 1: Net-(D37-Pad2) -> (no net)
- SWm1 pad 2: Columna7 -> (no net)
- SWn1 pad 1: Net-(D33-Pad2) -> (no net)
- SWn1 pad 2: Columna8 -> (no net)
- SWo1 pad 1: Net-(D43-Pad2) -> (no net)
- SWo1 pad 2: Columna6 -> (no net)
- SWp1 pad 1: Net-(D47-Pad2) -> (no net)
- SWp1 pad 2: Columna5 -> (no net)
- SWpgdown1 pad 1: Net-(D67-Pad2) -> (no net)
- SWpgdown1 pad 2: Columna16 -> (no net)
- SWpgup1 pad 1: Net-(D66-Pad2) -> (no net)
- SWpgup1 pad 2: Columna16 -> (no net)
- SWpunto1 pad 1: Net-(D45-Pad2) -> (no net)
- SWpunto1 pad 2: Columna5 -> (no net)
- SWshiftright1 pad 1: Net-(D57-Pad2) -> (no net)
- SWshiftright1 pad 2: Columna3 -> (no net)
- SWsigno1 pad 1: Net-(D54-Pad2) -> (no net)
- SWsigno1 pad 2: Columna3 -> (no net)
- SWu1 pad 1: Net-(D35-Pad2) -> (no net)
- SWu1 pad 2: Columna8 -> (no net)
- SW{1 pad 1: Net-(D53-Pad2) -> (no net)
- SW{1 pad 2: Columna4 -> (no net)
- SW}1 pad 1: Net-(D56-Pad2) -> (no net)
- SW}1 pad 2: Columna3 -> (no net)
Routing:
- net (no net): track 0.00 -> 5389.8 mm, vias 0 -> 94
- net GND: track 2066.8 -> 1190.1 mm, vias 3 -> 15
- net VCC: track 1973.2 -> 1118.2 mm, vias 1 -> 0
- net Fila5: track 681.1 -> 428.4 mm, vias 6 -> 2
- net Fila1: track 516.1 -> 282.7 mm
- net Fila3: track 579.8 -> 347.4 mm
- net Columna16: track 338.4 -> 108.9 mm, vias 6 -> 0
- net Fila6: track 528.8 -> 306.2 mm
- net Columna2: track 274.9 -> 102.5 mm, vias 6 -> 0
- net Columna3: track 259.0 -> 99.5 mm, vias 10 -> 0
- net Columna5: track 265.4 -> 108.2 mm, vias 8 -> 0
- net Columna4: track 249.2 -> 100.3 mm, vias 8 -> 0
- net Columna6: track 229.3 -> 101.3 mm, vias 8 -> 0
- net Columna8: track 225.6 -> 105.6 mm, vias 8 -> 0
- net Columna7: track 210.9 -> 91.5 mm, vias 9 -> 0
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- added copper zone on B.Cu, net GND
- added copper zone on F.Cu, net GND
Other:
- board size 3.6 x 3.1 mm -> 388.1 x 157.2 mm
