File: cuarenta/cuarenta.sch (KiCad schematic (older format))
At the start: 140 parts, among them J1 LED, SW1 SW_Push, SW10 SW_Push, SW11 SW_Push, SW12 SW_Push, SW13 SW_Push, SW14 SW_Push, SW15 SW_Push, SW16 SW_Push, SW17 SW_Push, SW18 SW_Push, SW19 SW_Push, SW2 SW_Push, SW20 SW_Push, SW21 SW_Push, SW22 SW_Push, SW23 SW_Push, SW25 SW_Push, SW26 SW_Push, SW27 SW_Push, SW29 SW_Push, SW3 SW_Push, SW30 SW_Push, SW31 SW_Push, SW33 SW_Push, SW34 SW_Push, SW35 SW_Push, SW36 SW_Push, SW37 SW_Push, SW38 SW_Push, SW39 SW_Push, SW4 SW_Push, SW40 SW_Push, SW41 SW_Push, SW42 SW_Push, SW43 SW_Push, SW44 SW_Push, SW45 SW_Push, SW46 SW_Push, SW47 SW_Push, SW48 SW_Push, SW49 Rotary_Encoder_Switch, SW5 SW_Push, SW6 SW_Push, SW7 SW_Push, SW8 SW_Push, SW9 SW_Push, U1 ARDUINO_MICRO_SHIELD

Commit message: Agregado 40%
Connections:
- net Row0: now also U1.A1; no longer U1.A2
- net Row1: now also U1.A2; no longer U1.A3
- net Row2: now also U1.A3; no longer U1.A4
- net Row3: now also U1.A4; no longer D49.1 (K), U1.A5
- new net Row4: D49.1 (K), U1.A5
- no-connect marks 9 -> 8
Changed lines of the file:
@@
 NoConn ~ 8750 3750
 NoConn ~ 8750 3650
-NoConn ~ 8750 2650
 NoConn ~ 8750 2550
 NoConn ~ 8750 2450
@@
 	1    0    0    -1
 $EndComp
-$Comp
-L mech7:power_GND #PWR0104
-U 1 1 612D41F2
-P -9150 1450
-F 0 "#PWR0104" H -9150 1200 50  0001 C CNN
-F 1 "power_GND" H -9145 1277 50  0000 C CNN
-F 2 "" H -9150 1450 50  0001 C CNN
-F 3 "" H -9150 1450 50  0001 C CNN
-	1    -9150 1450
-	1    0    0    -1
-$EndComp
 Text GLabel -9200 1150 0    50   Input ~ 0
 LED
@@
 	-1   0    0    -1
 $EndComp
-$Comp
-L mech7:power_GND #PWR0106
-U 1 1 613B89A7
-P -400 2550
-F 0 "#PWR0106" H -400 2300 50  0001 C CNN
-F 1 "power_GND" H -395 2377 50  0000 C CNN
-F 2 "" H -400 2550 50  0001 C CNN
-F 3 "" H -400 2550 50  0001 C CNN
-	1    -400 2550
-	-1   0    0    -1
-$EndComp
 Wire Wire Line
 	-650 2550 -400 2550
@@
 	1    0    0    -1
 $EndComp
-$Comp
-L mech7:power_GND #PWR0108
-U 1 1 613C9154
-P -9150 3550
-F 0 "#PWR0108" H -9150 3300 50  0001 C CNN
-F 1 "power_GND" H -9145 3377 50  0000 C CNN
-F 2 "" H -9150 3550 50  0001 C CNN
-F 3 "" H -9150 3550 50  0001 C CNN
-	1    -9150 3550
-	1    0    0    -1
-$EndComp
 Wire Wire Line
 	-8900 3550 -9150 3550
@@
 	-1   0    0    -1
 $EndComp
-$Comp
-L mech7:power_GND #PWR0110
-U 1 1 613DDB87
-P -400 4550
-F 0 "#PWR0110" H -400 4300 50  0001 C CNN
-F 1 "power_GND" H -395 4377 50  0000 C CNN
-F 2 "" H -400 4550 50  0001 C CNN
-F 3 "" H -400 4550 50  0001 C CNN
-	1    -400 4550
-	-1   0    0    -1
-$EndComp
 Wire Wire Line
 	-650 4550 -400 4550
@@
 Connection ~ 6050 4450
 Wire Wire Line
-	8400 1650 8400 4450
-Wire Wire Line
-	8400 4450 7850 4450
-Connection ~ 7850 4450
-Wire Wire Line
 	-9150 850  -8900 850
 Wire Wire Line
@@
 	3050 4450 4850 4450
 NoConn ~ 8750 3450
+Text GLabel 8750 2650 0    50   Input ~ 0
+Row0
+Text GLabel 8750 2950 0    50   Input ~ 0
+Row3
+Text GLabel 8750 2850 0    50   Input ~ 0
+Row2
 Text GLabel 8750 2750 0    50   Input ~ 0
-Row0
+Row1
 Text GLabel 8750 3050 0    50   Input ~ 0
-Row3
-Text GLabel 8750 2950 0    50   Input ~ 0
-Row2
-Text GLabel 8750 2850 0    50   Input ~ 0
-Row1
+Row4
+Text GLabel 8400 1650 3    50   Input ~ 0
+Row4
+$Comp
+L power:GND #PWR?
+U 1 1 6140EDFB
+P -400 2550
+F 0 "#PWR?" H -400 2300 50  0001 C CNN
+F 1 "GND" H -395 2377 50  0000 C CNN
+F 2 "" H -400 2550 50  0001 C CNN
+F 3 "" H -400 2550 50  0001 C CNN
+	1    -400 2550
+	1    0    0    -1
+$EndComp
+$Comp
+L power:GND #PWR?
+U 1 1 6143A185
+P -9150 1450
+F 0 "#PWR?" H -9150 1200 50  0001 C CNN
+F 1 "GND" H -9145 1277 50  0000 C CNN
+F 2 "" H -9150 1450 50  0001 C CNN
+F 3 "" H -9150 1450 50  0001 C CNN
+	1    -9150 1450
+	1    0    0    -1
+$EndComp
+$Comp
+L power:GND #PWR?
+U 1 1 6144F63F
+P -9150 3550
+F 0 "#PWR?" H -9150 3300 50  0001 C CNN
+F 1 "GND" H -9145 3377 50  0000 C CNN
+F 2 "" H -9150 3550 50  0001 C CNN
+F 3 "" H -9150 3550 50  0001 C CNN
+	1    -9150 3550
+	1    0    0    -1
+$EndComp
+$Comp
+L power:GND #PWR?
+U 1 1 614CF2EA
+P -400 4550
+F 0 "#PWR?" H -400 4300 50  0001 C CNN
+F 1 "GND" H -395 4377 50  0000 C CNN
+F 2 "" H -400 4550 50  0001 C CNN
+F 3 "" H -400 4550 50  0001 C CNN
+	1    -400 4550
+	1    0    0    -1
+$EndComp
 $EndSCHEMATC
