File: cuarenta/cuarenta.kicad_pcb (KiCad board)
At the start: 2 copper layers, 269.9 x 84.9 mm, 140 parts, among them J1 LED, SW1 SW_Push, SW10 SW_Push, SW11 SW_Push, SW12 SW_Push, SW13 SW_Push, SW14 SW_Push, SW15 SW_Push, SW16 SW_Push, SW17 SW_Push, SW18 SW_Push, SW19 SW_Push, SW2 SW_Push, SW20 SW_Push, SW21 SW_Push, SW22 SW_Push, SW23 SW_Push, SW25 SW_Push, SW26 SW_Push, SW27 SW_Push, SW29 SW_Push, SW3 SW_Push, SW30 SW_Push, SW31 SW_Push, SW33 SW_Push, SW34 SW_Push, SW35 SW_Push, SW36 SW_Push, SW37 SW_Push, SW38 SW_Push, SW39 SW_Push, SW4 SW_Push, SW40 SW_Push, SW41 SW_Push, SW42 SW_Push, SW43 SW_Push, SW44 SW_Push, SW45 SW_Push, SW46 SW_Push, SW47 SW_Push, SW48 SW_Push, SW49 Rotary_Encoder_Switch, SW5 SW_Push, SW6 SW_Push, SW7 SW_Push, SW8 SW_Push, SW9 SW_Push, U1 ARDUINO_MICRO_SHIELD

Commit message: Agregado 40%
Parts:
- removed D1, D10, D11, D12, D13, D14, D15, D16, D17, D18, D19, D2, D20, D21, D22, D23, D25, D26, D27, D29, D3, D30, D31, D33, D34, D35, D36, D37, D38, D39, D4, D40, D41, D42, D43, D44, D45, D46, D47, D48, D49, D5, D6, D7, D8, D9: 1N4148, Diode_THT:D_DO-35_SOD27_P7.62mm_Horizontal
- removed J1: LED, Mech1:StripLED_1side
- removed OL1: OLED, Mech0:OLED
- removed SW1, SW10, SW11, SW12, SW13, SW14, SW15, SW16, SW17, SW18, SW19, SW2, SW20, SW21, SW22, SW23, SW25, SW26, SW27, SW29, SW3, SW30, SW31, SW33, SW34, SW35, SW36, SW37, SW38, SW39, SW4, SW40, SW41, SW42, SW43, SW44, SW45, SW46, SW47, SW48, SW5, SW6, SW7, SW8, SW9: SW_Push, Mech0:CherryMX_Hotswap
- removed SW49: Rotary_Encoder_Switch, Mech0:RotaryEncoder_EC11
- removed U1: ARDUINO_MICRO_SHIELD, Mech6:ARDUINO_MICRO_SHIELD
- removed e1, e10, e11, e13, e14, e15, e16, e17, e18, e19, e2, e20, e21, e22, e23, e24, e25, e26, e27, e28, e29, e3, e30, e31, e32, e33, e34, e35, e36, e37, e38, e39, e40, e41, e42, e43, e44, e45, e46, e47, e48, e5, e6, e7, e9: e, Mech0:YS-SK6812MINI-E_2
- added REF**: case_cut, Mech0:case_cut, F.Cu at (78.4, 37.7)
- added REF**: case_cut, Mech0:case_cut, F.Cu at (226.0, 94.9)
- added REF**: case_cut, Mech0:case_cut, F.Cu at (245.1, 94.9)
- added REF**: case_cut, Mech0:case_cut, F.Cu at (264.1, 94.9)
- added REF**: case_cut, Mech0:case_cut, F.Cu at (264.1, 75.8)
- added REF**: case_cut, Mech0:case_cut, F.Cu at (245.1, 75.8)
- added REF**: case_cut, Mech0:case_cut, F.Cu at (226.0, 75.8)
- added REF**: case_cut, Mech0:case_cut, F.Cu at (207.0, 75.8)
- added REF**: case_cut, Mech0:case_cut, F.Cu at (187.9, 75.8)
- added REF**: case_cut, Mech0:case_cut, F.Cu at (168.9, 75.8)
- added REF**: case_cut, Mech0:case_cut, F.Cu at (149.8, 75.8)
- added REF** (x2): case_cut, Mech0:case_cut, F.Cu at (59.3, 37.7)
- added REF**: case_cut, Mech0:case_cut, F.Cu at (130.8, 75.8)
- added REF**: case_cut, Mech0:case_cut, F.Cu at (111.7, 75.8)
- added REF**: case_cut, Mech0:case_cut, F.Cu at (92.7, 75.8)
- added REF**: case_cut, Mech0:case_cut, F.Cu at (73.6, 75.8)
- added REF**: case_cut, Mech0:case_cut, F.Cu at (47.4, 75.8)
- added REF**: case_cut, Mech0:case_cut, F.Cu at (42.7, 56.8)
- added REF**: case_cut, Mech0:case_cut, F.Cu at (64.1, 56.8)
- added REF**: case_cut, Mech0:case_cut, F.Cu at (83.1, 56.8)
- added REF**: case_cut, Mech0:case_cut, F.Cu at (102.2, 56.8)
- added REF**: case_cut, Mech0:case_cut, F.Cu at (121.2, 56.8)
- added REF**: case_cut, Mech0:case_cut, F.Cu at (40.3, 37.7)
- added REF**: case_cut, Mech0:case_cut, F.Cu at (140.3, 56.8)
- added REF**: case_cut, Mech0:case_cut, F.Cu at (159.3, 56.8)
- added REF**: case_cut, Mech0:case_cut, F.Cu at (178.4, 56.8)
- added REF**: case_cut, Mech0:case_cut, F.Cu at (197.4, 56.8)
- added REF**: case_cut, Mech0:case_cut, F.Cu at (216.5, 56.8)
- added REF**: case_cut, Mech0:case_cut, F.Cu at (235.5, 56.8)
- added REF**: case_cut, Mech0:case_cut, F.Cu at (259.3, 56.8)
- added REF**: case_cut, Mech0:case_cut, F.Cu at (257.0, 37.7)
- added REF**: case_cut, Mech0:case_cut, F.Cu at (230.8, 37.7)
- added REF**: case_cut, Mech0:case_cut, F.Cu at (211.7, 37.7)
- added REF**: case_cut, Mech0:case_cut, F.Cu at (42.7, 94.9)
- added REF**: case_cut, Mech0:case_cut, F.Cu at (192.7, 37.7)
- added REF** (x2): case_cut, Mech0:case_cut, F.Cu at (97.4, 37.7)
- added REF** (x2): case_cut, Mech0:case_cut, F.Cu at (116.5, 37.7)
- added REF** (x2): case_cut, Mech0:case_cut, F.Cu at (135.5, 37.7)
- added REF** (x2): case_cut, Mech0:case_cut, F.Cu at (154.6, 37.7)
- added REF**: case_cut, Mech0:case_cut, F.Cu at (173.6, 37.7)
- added REF**: case_cut, Mech0:case_cut, F.Cu at (68.8, 94.9)
- added REF**: case_cut, Mech0:case_cut, F.Cu at (95.0, 94.9)
- added REF**: case_cut, Mech0:case_cut, F.Cu at (128.4, 94.9)
- added REF**: case_cut, Mech0:case_cut, F.Cu at (168.9, 94.9)
- added REF**: case_cut, Mech0:case_cut, F.Cu at (202.2, 94.9)
Routing:
- net GND: track 1153.4 -> 0.00 mm, vias 12 -> 0
- net VCC: track 1153.3 -> 0.00 mm
- net Row0: track 657.6 -> 0.00 mm
- net Row1: track 622.8 -> 0.00 mm
- net Row2: track 607.5 -> 0.00 mm
- net Row3: track 339.3 -> 0.00 mm
- net Col0: track 306.2 -> 0.00 mm, vias 6 -> 0
- net Col1: track 291.6 -> 0.00 mm, vias 6 -> 0
- net Col2: track 270.5 -> 0.00 mm, vias 6 -> 0
- net Col3: track 262.3 -> 0.00 mm, vias 6 -> 0
- net Col4: track 216.5 -> 0.00 mm, vias 4 -> 0
- net Col6: track 205.1 -> 0.00 mm, vias 6 -> 0
- net Col5: track 199.5 -> 0.00 mm, vias 4 -> 0
- net Col9: track 176.5 -> 0.00 mm, vias 6 -> 0
- net Col8: track 170.4 -> 0.00 mm, vias 6 -> 0
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- removed copper zone on B.Cu, net GND
- removed copper zone on F.Cu, net GND
Other:
- board size 269.9 x 84.9 mm -> 276 x 90.9 mm

Commit message: restaurados archivos 40%
Parts:
- removed REF** (x50): case_cut, Mech0:case_cut
- added D1: 1N4148, Diode_THT:D_DO-35_SOD27_P7.62mm_Horizontal, F.Cu at (24.8, 27.4)
- added D10: 1N4148, Diode_THT:D_DO-35_SOD27_P7.62mm_Horizontal, B.Cu at (67.6, 46.4)
- added D11: 1N4148, Diode_THT:D_DO-35_SOD27_P7.62mm_Horizontal, B.Cu at (77.1, 65.4)
- added D12: 1N4148, Diode_THT:D_DO-35_SOD27_P7.62mm_Horizontal, B.Cu at (79.4, 84.6)
- added D13: 1N4148, Diode_THT:D_DO-35_SOD27_P7.62mm_Horizontal, F.Cu at (81.8, 27.4)
- added D14: 1N4148, Diode_THT:D_DO-35_SOD27_P7.62mm_Horizontal, B.Cu at (86.6, 46.4)
- added D15: 1N4148, Diode_THT:D_DO-35_SOD27_P7.62mm_Horizontal, B.Cu at (96.1, 65.4)
- added D16: 1N4148, Diode_THT:D_DO-35_SOD27_P7.62mm_Horizontal, B.Cu at (112.8, 84.6)
- added D17: 1N4148, Diode_THT:D_DO-35_SOD27_P7.62mm_Horizontal, F.Cu at (100.8, 27.4)
- added D18: 1N4148, Diode_THT:D_DO-35_SOD27_P7.62mm_Horizontal, B.Cu at (105.8, 46.4)
- added D19: 1N4148, Diode_THT:D_DO-35_SOD27_P7.62mm_Horizontal, B.Cu at (115.1, 65.4)
- added D2: 1N4148, Diode_THT:D_DO-35_SOD27_P7.62mm_Horizontal, B.Cu at (27.1, 46.5)
- added D20: 1N4148, Diode_THT:D_DO-35_SOD27_P7.62mm_Horizontal, B.Cu at (153.3, 84.6)
- added D21: 1N4148, Diode_THT:D_DO-35_SOD27_P7.62mm_Horizontal, F.Cu at (120.0, 27.4)
- added D22: 1N4148, Diode_THT:D_DO-35_SOD27_P7.62mm_Horizontal, B.Cu at (124.8, 46.4)
- added D23: 1N4148, Diode_THT:D_DO-35_SOD27_P7.62mm_Horizontal, B.Cu at (134.3, 65.4)
- added D25: 1N4148, Diode_THT:D_DO-35_SOD27_P7.62mm_Horizontal, F.Cu at (139.0, 27.4)
- added D26: 1N4148, Diode_THT:D_DO-35_SOD27_P7.62mm_Horizontal, B.Cu at (143.8, 46.4)
- added D27: 1N4148, Diode_THT:D_DO-35_SOD27_P7.62mm_Horizontal, B.Cu at (153.3, 65.4)
- added D29: 1N4148, Diode_THT:D_DO-35_SOD27_P7.62mm_Horizontal, F.Cu at (158.0, 27.4)
- added D3: 1N4148, Diode_THT:D_DO-35_SOD27_P7.62mm_Horizontal, B.Cu at (31.8, 65.5)
- added D30: 1N4148, Diode_THT:D_DO-35_SOD27_P7.62mm_Horizontal, B.Cu at (162.8, 46.4)
- added D31: 1N4148, Diode_THT:D_DO-35_SOD27_P7.62mm_Horizontal, B.Cu at (172.3, 65.4)
- added D33: 1N4148, Diode_THT:D_DO-35_SOD27_P7.62mm_Horizontal, F.Cu at (177.2, 27.4)
- added D34: 1N4148, Diode_THT:D_DO-35_SOD27_P7.62mm_Horizontal, B.Cu at (182.0, 46.4)
- added D35: 1N4148, Diode_THT:D_DO-35_SOD27_P7.62mm_Horizontal, B.Cu at (191.3, 65.4)
- added D36: 1N4148, Diode_THT:D_DO-35_SOD27_P7.62mm_Horizontal, B.Cu at (186.6, 84.6)
- added D37: 1N4148, Diode_THT:D_DO-35_SOD27_P7.62mm_Horizontal, F.Cu at (196.2, 27.4)
- added D38: 1N4148, Diode_THT:D_DO-35_SOD27_P7.62mm_Horizontal, B.Cu at (201.0, 46.4)
- added D39: 1N4148, Diode_THT:D_DO-35_SOD27_P7.62mm_Horizontal, B.Cu at (210.6, 65.4)
- added D4: 1N4148, Diode_THT:D_DO-35_SOD27_P7.62mm_Horizontal, B.Cu at (27.1, 84.6)
- added D40: 1N4148, Diode_THT:D_DO-35_SOD27_P7.62mm_Horizontal, B.Cu at (210.4, 84.6)
- added D41: 1N4148, Diode_THT:D_DO-35_SOD27_P7.62mm_Horizontal, F.Cu at (215.2, 27.4)
- added D42: 1N4148, Diode_THT:D_DO-35_SOD27_P7.62mm_Horizontal, B.Cu at (220.0, 46.4)
- added D43: 1N4148, Diode_THT:D_DO-35_SOD27_P7.62mm_Horizontal, B.Cu at (229.6, 65.4)
- added D44: 1N4148, Diode_THT:D_DO-35_SOD27_P7.62mm_Horizontal, B.Cu at (229.6, 84.4)
- added D45: 1N4148, Diode_THT:D_DO-35_SOD27_P7.62mm_Horizontal, F.Cu at (241.4, 27.4)
- added D46: 1N4148, Diode_THT:D_DO-35_SOD27_P7.62mm_Horizontal, B.Cu at (243.8, 46.5)
- added D47: 1N4148, Diode_THT:D_DO-35_SOD27_P7.62mm_Horizontal, B.Cu at (248.6, 65.4)
- added D48: 1N4148, Diode_THT:D_DO-35_SOD27_P7.62mm_Horizontal, B.Cu at (248.6, 84.4)
- added D49: 1N4148, Diode_THT:D_DO-35_SOD27_P7.62mm_Horizontal, B.Cu at (267.9, 100.1)
- added D5: 1N4148, Diode_THT:D_DO-35_SOD27_P7.62mm_Horizontal, F.Cu at (43.8, 27.4)
- added D6: 1N4148, Diode_THT:D_DO-35_SOD27_P7.62mm_Horizontal, B.Cu at (48.6, 46.4)
- added D7: 1N4148, Diode_THT:D_DO-35_SOD27_P7.62mm_Horizontal, B.Cu at (58.1, 65.4)
- added D8: 1N4148, Diode_THT:D_DO-35_SOD27_P7.62mm_Horizontal, B.Cu at (53.2, 84.6)
- added D9: 1N4148, Diode_THT:D_DO-35_SOD27_P7.62mm_Horizontal, F.Cu at (62.8, 27.4)
- added J1: LED, Mech1:StripLED_1side, B.Cu at (260.9, 82.0)
- added OL1: OLED, Mech0:OLED, F.Cu at (267.1, 76.3)
- added SW1: SW_Push, Mech0:CherryMX_Hotswap, F.Cu at (24.2, 35.8)
- added SW10: SW_Push, Mech0:CherryMX_Hotswap, F.Cu at (67.1, 54.9)
- added SW11: SW_Push, Mech0:CherryMX_Hotswap, F.Cu at (76.6, 73.9)
- added SW12: SW_Push, Mech0:CherryMX_Hotswap, F.Cu at (79.0, 93.0)
- added SW13: SW_Push, Mech0:CherryMX_Hotswap, F.Cu at (81.3, 35.8)
- added SW14: SW_Push, Mech0:CherryMX_Hotswap, F.Cu at (86.1, 54.9)
- added SW15: SW_Push, Mech0:CherryMX_Hotswap, F.Cu at (95.6, 73.9)
- added SW16: SW_Push, Mech0:CherryMX_Hotswap, F.Cu at (112.3, 93.0)
- added SW17: SW_Push, Mech0:CherryMX_Hotswap, F.Cu at (100.4, 35.8)
- added SW18: SW_Push, Mech0:CherryMX_Hotswap, F.Cu at (105.2, 54.9)
- added SW19: SW_Push, Mech0:CherryMX_Hotswap, F.Cu at (114.7, 73.9)
- added SW2: SW_Push, Mech0:CherryMX_Hotswap, F.Cu at (26.6, 54.9)
- added SW20: SW_Push, Mech0:CherryMX_Hotswap, F.Cu at (152.8, 93.0)
- added SW21: SW_Push, Mech0:CherryMX_Hotswap, F.Cu at (119.4, 35.8)
- added SW22: SW_Push, Mech0:CherryMX_Hotswap, F.Cu at (124.2, 54.9)
- added SW23: SW_Push, Mech0:CherryMX_Hotswap, F.Cu at (133.7, 73.9)
- added SW25: SW_Push, Mech0:CherryMX_Hotswap, F.Cu at (138.5, 35.8)
- added SW26: SW_Push, Mech0:CherryMX_Hotswap, F.Cu at (143.3, 54.9)
- added SW27: SW_Push, Mech0:CherryMX_Hotswap, F.Cu at (152.8, 73.9)
- added SW29: SW_Push, Mech0:CherryMX_Hotswap, F.Cu at (157.5, 35.8)
- added SW3: SW_Push, Mech0:CherryMX_Hotswap, F.Cu at (31.3, 73.9)
- added SW30: SW_Push, Mech0:CherryMX_Hotswap, F.Cu at (162.3, 54.9)
- added SW31: SW_Push, Mech0:CherryMX_Hotswap, F.Cu at (171.8, 73.9)
- added SW33: SW_Push, Mech0:CherryMX_Hotswap, F.Cu at (176.6, 35.8)
- added SW34: SW_Push, Mech0:CherryMX_Hotswap, F.Cu at (181.4, 54.9)
- added SW35: SW_Push, Mech0:CherryMX_Hotswap, F.Cu at (190.9, 73.9)
- added SW36: SW_Push, Mech0:CherryMX_Hotswap, F.Cu at (186.1, 93.0)
- added SW37: SW_Push, Mech0:CherryMX_Hotswap, F.Cu at (195.6, 35.8)
- added SW38: SW_Push, Mech0:CherryMX_Hotswap, F.Cu at (200.4, 54.9)
- added SW39: SW_Push, Mech0:CherryMX_Hotswap, F.Cu at (209.9, 73.9)
- added SW4: SW_Push, Mech0:CherryMX_Hotswap, F.Cu at (26.6, 93.0)
- added SW40: SW_Push, Mech0:CherryMX_Hotswap, F.Cu at (209.9, 93.0)
- added SW41: SW_Push, Mech0:CherryMX_Hotswap, F.Cu at (214.7, 35.8)
- added SW42: SW_Push, Mech0:CherryMX_Hotswap, F.Cu at (219.5, 54.9)
- added SW43: SW_Push, Mech0:CherryMX_Hotswap, F.Cu at (229.0, 73.9)
- added SW44: SW_Push, Mech0:CherryMX_Hotswap, F.Cu at (229.0, 93.0)
- added SW45: SW_Push, Mech0:CherryMX_Hotswap, F.Cu at (240.9, 35.8)
- added SW46: SW_Push, Mech0:CherryMX_Hotswap, F.Cu at (243.3, 54.9)
- added SW47: SW_Push, Mech0:CherryMX_Hotswap, F.Cu at (248.0, 73.9)
- added SW48: SW_Push, Mech0:CherryMX_Hotswap, F.Cu at (248.0, 93.0)
- added SW49: Rotary_Encoder_Switch, Mech0:RotaryEncoder_EC11, F.Cu at (271.8, 90.6)
- added SW5: SW_Push, Mech0:CherryMX_Hotswap, F.Cu at (43.2, 35.8)
- added SW6: SW_Push, Mech0:CherryMX_Hotswap, F.Cu at (48.0, 54.9)
- added SW7: SW_Push, Mech0:CherryMX_Hotswap, F.Cu at (57.5, 73.9)
- added SW8: SW_Push, Mech0:CherryMX_Hotswap, F.Cu at (52.8, 93.0)
- added SW9: SW_Push, Mech0:CherryMX_Hotswap, F.Cu at (62.3, 35.8)
- added U1: ARDUINO_MICRO_SHIELD, Mech6:ARDUINO_MICRO_SHIELD, B.Cu at (262.5, 73.9)
- added e1: e, Mech0:YS-SK6812MINI-E_2, B.Cu at (24.2, 40.5)
- added e10: e, Mech0:YS-SK6812MINI-E_2, B.Cu at (67.1, 59.6)
- added e11: e, Mech0:YS-SK6812MINI-E_2, B.Cu at (76.6, 78.6)
- added e13: e, Mech0:YS-SK6812MINI-E_2, B.Cu at (81.3, 40.5)
- added e14: e, Mech0:YS-SK6812MINI-E_2, B.Cu at (86.1, 59.6)
- added e15: e, Mech0:YS-SK6812MINI-E_2, B.Cu at (95.6, 78.6)
- added e16: e, Mech0:YS-SK6812MINI-E_2, B.Cu at (26.6, 97.7)
- added e17: e, Mech0:YS-SK6812MINI-E_2, B.Cu at (100.4, 40.5)
- added e18: e, Mech0:YS-SK6812MINI-E_2, B.Cu at (105.2, 59.6)
- added e19: e, Mech0:YS-SK6812MINI-E_2, B.Cu at (114.7, 78.6)
- added e2: e, Mech0:YS-SK6812MINI-E_2, B.Cu at (26.6, 59.6)
- added e20: e, Mech0:YS-SK6812MINI-E_2, B.Cu at (52.8, 97.7)
- added e21: e, Mech0:YS-SK6812MINI-E_2, B.Cu at (119.4, 40.5)
- added e22: e, Mech0:YS-SK6812MINI-E_2, B.Cu at (124.2, 59.6)
- added e23: e, Mech0:YS-SK6812MINI-E_2, B.Cu at (133.7, 78.6)
- added e24: e, Mech0:YS-SK6812MINI-E_2, B.Cu at (79.0, 97.7)
- added e25: e, Mech0:YS-SK6812MINI-E_2, B.Cu at (138.5, 40.5)
- added e26: e, Mech0:YS-SK6812MINI-E_2, B.Cu at (143.3, 59.6)
- added e27: e, Mech0:YS-SK6812MINI-E_2, B.Cu at (152.8, 78.6)
- added e28: e, Mech0:YS-SK6812MINI-E_2, B.Cu at (112.3, 97.7)
- added e29: e, Mech0:YS-SK6812MINI-E_2, B.Cu at (157.5, 40.5)
- added e3: e, Mech0:YS-SK6812MINI-E_2, B.Cu at (31.3, 78.6)
- added e30: e, Mech0:YS-SK6812MINI-E_2, B.Cu at (162.3, 59.6)
- added e31: e, Mech0:YS-SK6812MINI-E_2, B.Cu at (171.8, 78.6)
- added e32: e, Mech0:YS-SK6812MINI-E_2, B.Cu at (152.8, 97.7)
- added e33: e, Mech0:YS-SK6812MINI-E_2, B.Cu at (176.6, 40.5)
- added e34: e, Mech0:YS-SK6812MINI-E_2, B.Cu at (181.4, 59.6)
- added e35: e, Mech0:YS-SK6812MINI-E_2, B.Cu at (190.9, 78.6)
- added e36: e, Mech0:YS-SK6812MINI-E_2, B.Cu at (186.1, 97.7)
- added e37: e, Mech0:YS-SK6812MINI-E_2, B.Cu at (195.6, 40.5)
- added e38: e, Mech0:YS-SK6812MINI-E_2, B.Cu at (200.4, 59.6)
- added e39: e, Mech0:YS-SK6812MINI-E_2, B.Cu at (209.9, 78.6)
- added e40: e, Mech0:YS-SK6812MINI-E_2, B.Cu at (209.9, 97.7)
- added e41: e, Mech0:YS-SK6812MINI-E_2, B.Cu at (214.7, 40.5)
- added e42: e, Mech0:YS-SK6812MINI-E_2, B.Cu at (219.5, 59.6)
- added e43: e, Mech0:YS-SK6812MINI-E_2, B.Cu at (229.0, 78.6)
- added e44: e, Mech0:YS-SK6812MINI-E_2, B.Cu at (229.0, 97.7)
- added e45: e, Mech0:YS-SK6812MINI-E_2, B.Cu at (240.9, 40.5)
- added e46: e, Mech0:YS-SK6812MINI-E_2, B.Cu at (243.3, 59.6)
- added e47: e, Mech0:YS-SK6812MINI-E_2, B.Cu at (248.0, 78.6)
- added e48: e, Mech0:YS-SK6812MINI-E_2, B.Cu at (248.0, 97.7)
- added e5: e, Mech0:YS-SK6812MINI-E_2, B.Cu at (43.2, 40.5)
- added e6: e, Mech0:YS-SK6812MINI-E_2, B.Cu at (48.0, 59.6)
- added e7: e, Mech0:YS-SK6812MINI-E_2, B.Cu at (57.5, 78.6)
- added e9: e, Mech0:YS-SK6812MINI-E_2, B.Cu at (62.3, 40.5)
Routing:
- net GND: track 0.00 -> 1153.4 mm, vias 0 -> 12
- net VCC: track 0.00 -> 1153.3 mm
- net Row0: track 0.00 -> 657.6 mm
- net Row1: track 0.00 -> 622.8 mm
- net Row2: track 0.00 -> 607.5 mm
- net Row3: track 0.00 -> 339.3 mm
- net Col0: track 0.00 -> 306.2 mm, vias 0 -> 6
- net Col1: track 0.00 -> 291.6 mm, vias 0 -> 6
- net Col2: track 0.00 -> 270.5 mm, vias 0 -> 6
- net Col3: track 0.00 -> 262.3 mm, vias 0 -> 6
- net Col4: track 0.00 -> 216.5 mm, vias 0 -> 4
- net Col6: track 0.00 -> 205.1 mm, vias 0 -> 6
- net Col5: track 0.00 -> 199.5 mm, vias 0 -> 4
- net Col9: track 0.00 -> 176.5 mm, vias 0 -> 6
- net Col8: track 0.00 -> 170.4 mm, vias 0 -> 6
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- added copper zone on B.Cu, net GND
- added copper zone on F.Cu, net GND
Other:
- board size 276 x 90.9 mm -> 269.9 x 84.9 mm
- net class Default removed
