File: 65%/stain/stain.kicad_sch (KiCad schematic)
At the start: 212 parts, among them J1 LED, SW1 Switch_SW_Push, SW10 Switch_SW_Push, SW11 Switch_SW_Push, SW12 Switch_SW_Push, SW13 Switch_SW_Push, SW14 Switch_SW_Push, SW15 Switch_SW_Push, SW16 Switch_SW_Push, SW17 Switch_SW_Push, SW18 Switch_SW_Push, SW19 Switch_SW_Push, SW2 Switch_SW_Push, SW20 Switch_SW_Push, SW21 Switch_SW_Push, SW22 Switch_SW_Push, SW23 Switch_SW_Push, SW24 Switch_SW_Push, SW25 Switch_SW_Push, SW26 Switch_SW_Push, SW27 Switch_SW_Push, SW28 Switch_SW_Push, SW29 Switch_SW_Push, SW3 Switch_SW_Push, SW30 Switch_SW_Push, SW31 Switch_SW_Push, SW32 Switch_SW_Push, SW33 Switch_SW_Push, SW34 Switch_SW_Push, SW35 Switch_SW_Push, SW36 Switch_SW_Push, SW37 Switch_SW_Push, SW38 Switch_SW_Push, SW39 Switch_SW_Push, SW4 Switch_SW_Push, SW40 Switch_SW_Push, SW41 Switch_SW_Push, SW42 Switch_SW_Push, SW43 Switch_SW_Push, SW44 Switch_SW_Push, SW45 Switch_SW_Push, SW46 Switch_SW_Push, SW47 Switch_SW_Push, SW48 Switch_SW_Push, SW49 Switch_SW_Push, SW5 Switch_SW_Push, SW50 Switch_SW_Push, SW51 Switch_SW_Push, SW52 Switch_SW_Push, SW53 Switch_SW_Push, SW54 Switch_SW_Push, SW55 Switch_SW_Push, SW56 Switch_SW_Push, SW57 Switch_SW_Push, SW58 Switch_SW_Push, SW59 Switch_SW_Push, SW6 Switch_SW_Push, SW60 Switch_SW_Push, SW61 Switch_SW_Push, SW62 Switch_SW_Push, SW63 Switch_SW_Push, SW64 Switch_SW_Push, SW65 Switch_SW_Push, SW66 Switch_SW_Push, SW67 Switch_SW_Push, SW68 Switch_SW_Push, SW69 Switch_SW_Push, SW7 Switch_SW_Push, SW70 Device_Rotary_Encoder_Switch, SW8 Switch_SW_Push, SW9 Switch_SW_Push, U1 ARDUINO_MICRO_SHIELD

Commit message: EndGame 30042023
Connections:
- net Col0: now also SW1.2, SW16.2, SW31.2, SW45.2, SW67.2, U1.A5; no longer U1.RX (0/RX)
- net Col1: now also SW17.2, SW2.2, SW32.2, SW46.2, SW68.2, U1.A4; no longer SW1.2, SW16.2, SW31.2, SW45.2, SW67.2, U1.12 (12/A11)
- net Col10: now also SW11.2, SW26.2, SW41.2, SW55.2, SW62.2, U1.4 (4/A6); no longer OL1.3 (SCL), SW10.2, SW25.2, SW40.2, SW54.2, SW61.2, U1.3 (3(PWM)/SCL)
- net Col11: now also OL1.3 (SCL), SW12.2, SW27.2, SW42.2, SW56.2, SW63.2, U1.3 (3(PWM)/SCL); no longer OL1.4 (SDA), SW11.2, SW26.2, SW41.2, SW55.2, SW62.2, U1.2 (2/SDA)
- net Col12: now also SW13.2, SW28.2, SW43.2, SW57.2, SW64.2, U1.MI (MISO); no longer SW12.2, SW27.2, SW42.2, SW56.2, SW63.2, U1.A4
- net Col13: now also SW14.2, SW44.2, SW58.2, SW65.2, U1.SCK; no longer SW13.2, SW28.2, SW43.2, SW57.2, SW64.2, U1.A5
- net Col14: now also OL1.4 (SDA), SW15.2, SW30.2, SW59.2, SW66.2, SW70.S2, U1.2 (2/SDA); no longer SW14.2, SW44.2, SW58.2, SW65.2, U1.MI (MISO)
- net Col15: now also D70.1 (K), U1.RX (0/RX); no longer SW15.2, SW30.2, SW59.2, SW66.2, SW70.S2, U1.SCK
- net Col2: now also SW18.2, SW3.2, SW33.2, SW47.2, SW69.2, U1.A3; no longer SW17.2, SW2.2, SW32.2, SW46.2, SW68.2, U1.11 (11(PWM))
- net Col3: now also SW19.2, SW34.2, SW4.2, SW48.2, U1.A2; no longer SW18.2, SW3.2, SW33.2, SW47.2, SW69.2, U1.10 (10(PWM)/A10)
- net Col4: now also SW20.2, SW35.2, SW49.2, SW5.2, U1.A1; no longer SW19.2, SW34.2, SW4.2, SW48.2, U1.9 (9(PWM)/A9)
- net Col5: now also SW21.2, SW36.2, SW50.2, SW6.2, U1.A0; no longer SW20.2, SW35.2, SW49.2, SW5.2, U1.8 (8/A8)
- net Col6: now also SW22.2, SW37.2, SW51.2, SW60.2, SW7.2, U1.13 (13(PWM)); no longer SW21.2, SW36.2, SW50.2, SW6.2, U1.7
- net Col7: now also SW23.2, SW38.2, SW52.2, SW8.2, U1.7; no longer SW22.2, SW37.2, SW51.2, SW60.2, SW7.2, U1.6 (6(PWM)/A7)
- net Col8: now also SW24.2, SW39.2, SW53.2, SW9.2, U1.6 (6(PWM)/A7); no longer SW23.2, SW38.2, SW52.2, SW8.2, U1.5 (5(PWM))
- net Col9: now also SW10.2, SW25.2, SW40.2, SW54.2, SW61.2, U1.5 (5(PWM)); no longer SW24.2, SW39.2, SW53.2, SW9.2, U1.4 (4/A6)
- net GND: now also LED16.3 (VSS), LED17.3 (VSS), LED18.3 (VSS), LED19.3 (VSS), LED20.3 (VSS), LED21.3 (VSS), LED22.3 (VSS), LED23.3 (VSS), LED24.3 (VSS), LED25.3 (VSS), LED26.3 (VSS), LED27.3 (VSS), LED28.3 (VSS), LED29.3 (VSS), LED30.3 (VSS), LED45.3 (VSS), LED46.3 (VSS), LED47.3 (VSS), LED48.3 (VSS), LED49.3 (VSS), LED50.3 (VSS), LED51.3 (VSS), LED52.3 (VSS), LED53.3 (VSS), LED54.3 (VSS), LED55.3 (VSS), LED56.3 (VSS), LED57.3 (VSS), LED58.3 (VSS), LED59.3 (VSS), LED60.3 (VSS), LED61.3 (VSS), LED62.3 (VSS), LED63.3 (VSS), LED64.3 (VSS), LED65.3 (VSS), LED66.3 (VSS), LED67.3 (VSS), LED68.3 (VSS), LED69.3 (VSS); no longer LED16.1 (VDD), LED17.1 (VDD), LED18.1 (VDD), LED19.1 (VDD), LED20.1 (VDD), LED21.1 (VDD), LED22.1 (VDD), LED23.1 (VDD), LED24.1 (VDD), LED25.1 (VDD), LED26.1 (VDD), LED27.1 (VDD), LED28.1 (VDD), LED29.1 (VDD), LED30.1 (VDD), LED45.1 (VDD), LED46.1 (VDD), LED47.1 (VDD), LED48.1 (VDD), LED49.1 (VDD), LED50.1 (VDD), LED51.1 (VDD), LED52.1 (VDD), LED53.1 (VDD), LED54.1 (VDD), LED55.1 (VDD), LED56.1 (VDD), LED57.1 (VDD), LED58.1 (VDD), LED59.1 (VDD), LED60.1 (VDD), LED61.1 (VDD), LED62.1 (VDD), LED63.1 (VDD), LED64.1 (VDD), LED65.1 (VDD), LED66.1 (VDD), LED67.1 (VDD), LED68.1 (VDD), LED69.1 (VDD)
- net LED: now also LED8.2 (DOUT); no longer LED9.4 (DIN)
- net Row1: now also U1.8 (8/A8); no longer U1.13 (13(PWM))
- net Row2: now also U1.9 (9(PWM)/A9); no longer D29.1 (K), U1.A0
- net Row3: now also D29.1 (K), U1.10 (10(PWM)/A10); no longer D70.1 (K), U1.A1
- net Row4: now also U1.11 (11(PWM)); no longer U1.A2
- net Row5: now also U1.12 (12/A11); no longer U1.A3
- net VCC: now also LED16.1 (VDD), LED17.1 (VDD), LED18.1 (VDD), LED19.1 (VDD), LED20.1 (VDD), LED21.1 (VDD), LED22.1 (VDD), LED23.1 (VDD), LED24.1 (VDD), LED25.1 (VDD), LED26.1 (VDD), LED27.1 (VDD), LED28.1 (VDD), LED29.1 (VDD), LED30.1 (VDD), LED45.1 (VDD), LED46.1 (VDD), LED47.1 (VDD), LED48.1 (VDD), LED49.1 (VDD), LED50.1 (VDD), LED51.1 (VDD), LED52.1 (VDD), LED53.1 (VDD), LED54.1 (VDD), LED55.1 (VDD), LED56.1 (VDD), LED57.1 (VDD), LED58.1 (VDD), LED59.1 (VDD), LED60.1 (VDD), LED61.1 (VDD), LED62.1 (VDD), LED63.1 (VDD), LED64.1 (VDD), LED65.1 (VDD), LED66.1 (VDD), LED67.1 (VDD), LED68.1 (VDD), LED69.1 (VDD); no longer LED16.3 (VSS), LED17.3 (VSS), LED18.3 (VSS), LED19.3 (VSS), LED20.3 (VSS), LED21.3 (VSS), LED22.3 (VSS), LED23.3 (VSS), LED24.3 (VSS), LED25.3 (VSS), LED26.3 (VSS), LED27.3 (VSS), LED28.3 (VSS), LED29.3 (VSS), LED30.3 (VSS), LED45.3 (VSS), LED46.3 (VSS), LED47.3 (VSS), LED48.3 (VSS), LED49.3 (VSS), LED50.3 (VSS), LED51.3 (VSS), LED52.3 (VSS), LED53.3 (VSS), LED54.3 (VSS), LED55.3 (VSS), LED56.3 (VSS), LED57.3 (VSS), LED58.3 (VSS), LED59.3 (VSS), LED60.3 (VSS), LED61.3 (VSS), LED62.3 (VSS), LED63.3 (VSS), LED64.3 (VSS), LED65.3 (VSS), LED66.3 (VSS), LED67.3 (VSS), LED68.3 (VSS), LED69.3 (VSS)
- net at LED56.2 (DOUT): now also LED55.4 (DIN); no longer LED57.4 (DIN)
- net at LED56.4 (DIN): now also LED57.2 (DOUT); no longer LED55.2 (DOUT)
- net at LED43.2 (DOUT): now also LED42.4 (DIN); no longer LED44.4 (DIN)
- net at LED43.4 (DIN): now also LED44.2 (DOUT); no longer LED42.2 (DOUT)
- net at LED59.2 (DOUT): now also LED58.4 (DIN); no longer LED31.4 (DIN)
- net at LED59.4 (DIN): now also LED69.2 (DOUT); no longer LED58.2 (DOUT)
- net at LED51.2 (DOUT): now also LED50.4 (DIN); no longer LED52.4 (DIN)
- net at LED51.4 (DIN): now also LED52.2 (DOUT); no longer LED50.2 (DOUT)
- net at LED18.2 (DOUT): now also LED17.4 (DIN); no longer LED19.4 (DIN)
- net at LED18.4 (DIN): now also LED19.2 (DOUT); no longer LED17.2 (DOUT)
- net at LED38.2 (DOUT): now also LED37.4 (DIN); no longer LED39.4 (DIN)
- net at LED38.4 (DIN): now also LED39.2 (DOUT); no longer LED37.2 (DOUT)
- net at LED31.2 (DOUT): now also LED16.4 (DIN); no longer LED32.4 (DIN)
- net at LED62.2 (DOUT): now also LED63.4 (DIN); no longer LED61.4 (DIN)
- net at LED62.4 (DIN): now also LED61.2 (DOUT); no longer LED63.2 (DOUT)
- net at LED40.2 (DOUT): now also LED39.4 (DIN); no longer LED41.4 (DIN)
- net at LED40.4 (DIN): now also LED41.2 (DOUT); no longer LED39.2 (DOUT)
- net at LED66.2 (DOUT): now also LED67.4 (DIN); no longer LED65.4 (DIN)
- net at LED66.4 (DIN): now also LED65.2 (DOUT); no longer LED67.2 (DOUT)
- net at LED20.4 (DIN): now also LED21.2 (DOUT); no longer LED19.2 (DOUT)
- net at LED36.2 (DOUT): now also LED35.4 (DIN); no longer LED37.4 (DIN)
- net at LED49.2 (DOUT): now also LED48.4 (DIN); no longer LED50.4 (DIN)
- net at LED49.4 (DIN): now also LED50.2 (DOUT); no longer LED48.2 (DOUT)
- net at LED30.2 (DOUT): now also LED29.4 (DIN); no longer LED16.4 (DIN)
- net at LED30.4 (DIN): now also LED16.2 (DOUT); no longer LED29.2 (DOUT)
- net at LED60.2 (DOUT): now also LED61.4 (DIN); no longer LED45.4 (DIN)
- net at LED60.4 (DIN): no longer LED61.2 (DOUT)
- net at LED53.2 (DOUT): now also LED52.4 (DIN); no longer LED54.4 (DIN)
- net at LED53.4 (DIN): now also LED54.2 (DOUT); no longer LED52.2 (DOUT)
- net at LED24.2 (DOUT): now also LED23.4 (DIN); no longer LED25.4 (DIN)
- net at LED24.4 (DIN): now also LED25.2 (DOUT); no longer LED23.2 (DOUT)
- net at LED64.4 (DIN): now also LED63.2 (DOUT); no longer LED65.2 (DOUT)
- net at LED28.2 (DOUT): now also LED27.4 (DIN); no longer LED29.4 (DIN)
- net at LED28.4 (DIN): now also LED29.2 (DOUT); no longer LED27.2 (DOUT)
- net at LED64.2 (DOUT): now also LED65.4 (DIN); no longer LED63.4 (DIN)
- net at LED22.2 (DOUT): now also LED21.4 (DIN); no longer LED23.4 (DIN)
- net at LED26.2 (DOUT): now also LED25.4 (DIN); no longer LED27.4 (DIN)
- net at LED45.2 (DOUT): now also LED44.4 (DIN); no longer LED46.4 (DIN)
- net at LED36.4 (DIN): now also LED37.2 (DOUT); no longer LED35.2 (DOUT)
- net at LED34.2 (DOUT): now also LED33.4 (DIN); no longer LED35.4 (DIN)
- net at LED34.4 (DIN): now also LED35.2 (DOUT); no longer LED33.2 (DOUT)
- net at LED26.4 (DIN): now also LED27.2 (DOUT); no longer LED25.2 (DOUT)
- net at LED68.2 (DOUT): now also LED69.4 (DIN); no longer LED67.4 (DIN)
- net at LED68.4 (DIN): now also LED67.2 (DOUT); no longer LED69.2 (DOUT)
- net at LED20.2 (DOUT): now also LED19.4 (DIN); no longer LED21.4 (DIN)
- net at LED47.2 (DOUT): now also LED46.4 (DIN); no longer LED48.4 (DIN)
- net at LED46.2 (DOUT): now also LED45.4 (DIN); no longer LED47.4 (DIN)
- net at LED22.4 (DIN): now also LED23.2 (DOUT); no longer LED21.2 (DOUT)
- net at LED32.2 (DOUT): now also LED31.4 (DIN); no longer LED33.4 (DIN)
- new net: LED17.2 (DOUT), LED9.4 (DIN)
- new net: LED57.4 (DIN), LED58.2 (DOUT)
- new net: LED41.4 (DIN), LED42.2 (DOUT)
- new net: LED54.4 (DIN), LED55.2 (DOUT)
- new net: LED47.4 (DIN), LED48.2 (DOUT)
- new net: LED32.4 (DIN), LED33.2 (DOUT)
- no-connect marks 0 -> 5
Other:
- moved on the sheet: D1, D10, D11, D12, D13, D14, D15, D16, D17, D18, D19, D2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
