File: EndGame/EndGame/EndGame.kicad_sch (KiCad schematic)
At the start: 4 parts

Commit message: 24092024
Parts:
- removed U?: ARDUINO_MICRO_SHIELD, symbol Meca0:ARDUINO_MICRO_SHIELD
- added D1, D10, D11, D12, D13, D14, D15, D16, D17, D18, D19, D2, D20, D21, D22, D23, D24, D25, D26, D27, D28, D29, D3, D30, D31, D32, D33, D34, D35, D36, D37, D38, D39, D4, D40, D41, D42, D43, D44, D45, D46, D47, D48, D49, D5, D50, D51, D52, D53, D54, D55, D56, D57, D58, D59, D6, D60, D61, D62, D63, D64, D65, D66, D67, D68, D69, D7, D70, D71, D72, D73, D74, D75, D76, D77, D8, D9: Diode_1N4148, Diode_THT:D_DO-35_SOD27_P7.62mm_Horizontal, symbol 1i_SplitKeyboard-cache:Diode_1N4148
- added LED1, LED10, LED11, LED12, LED13, LED14, LED15, LED16, LED17, LED18, LED19, LED2, LED20, LED21, LED22, LED23, LED24, LED25, LED26, LED27, LED28, LED29, LED3, LED30, LED31, LED32, LED33, LED34, LED35, LED36, LED37, LED38, LED39, LED4, LED40, LED41, LED42, LED43, LED44, LED45, LED46, LED47, LED48, LED49, LED5, LED50, LED51, LED52, LED53, LED54, LED55, LED56, LED57, LED58, LED59, LED6, LED60, LED61, LED62, LED63, LED64, LED65, LED66, LED67, LED68, LED69, LED7, LED70, LED71, LED72, LED73, LED74, LED75, LED76, LED8, LED9: YS-SK6812, cherry:YS-SK6812MINI-E_2, symbol kicad:Mech_4_YS-SK6812MINI-E
- added SW1, SW10, SW11, SW12, SW13, SW14, SW15, SW16, SW17, SW18, SW19, SW2, SW20, SW21, SW22, SW23, SW24, SW25, SW26, SW27, SW28, SW29, SW3, SW30, SW31, SW32, SW33, SW34, SW35, SW36, SW37, SW38, SW39, SW4, SW40, SW41, SW42, SW43, SW44, SW45, SW46, SW47, SW48, SW49, SW5, SW50, SW51, SW52, SW53, SW54, SW55, SW56, SW57, SW58, SW59, SW6, SW60, SW61, SW62, SW63, SW64, SW65, SW66, SW67, SW68, SW69, SW7, SW70, SW71, SW72, SW73, SW74, SW75, SW76, SW8, SW9: SW_PUSH, cherry:CherryMX_Hotswap, symbol 1i_SplitKeyboard-cache:Switch_SW_Push
- added U2: Mech_8_ARDUINO_MICRO_SHIELD, cherry:ARDUINO_MICRO_SHIELD, symbol kicad:Mech_8_ARDUINO_MICRO_SHIELD
- J1: renamed from J?; footprint Meca:StripLED_1side -> cherry:StripLED_1side
- OL1: renamed from OL?; footprint (none) -> cherry:OLED_v2
- SW77: renamed from SW?; footprint (none) -> cherry:RotaryEncoder_EC11
Connections:
- net GND: now reaches OL1.1 (GND)
- net GND: now also J1.3 (GND), SW77.C, LED1.3 (VSS), LED10.3 (VSS), LED11.3 (VSS), LED12.3 (VSS), LED13.3 (VSS), LED14.3 (VSS), LED15.3 (VSS), LED16.3 (VSS), LED17.3 (VSS), LED18.3 (VSS), LED19.3 (VSS), LED2.3 (VSS), LED20.3 (VSS), LED21.3 (VSS), LED22.3 (VSS), LED23.3 (VSS), LED24.3 (VSS), LED25.3 (VSS), LED26.3 (VSS), LED27.3 (VSS), LED28.3 (VSS), LED29.3 (VSS), LED3.3 (VSS), LED30.3 (VSS), LED31.3 (VSS), LED32.3 (VSS), LED33.3 (VSS), LED34.3 (VSS), LED35.3 (VSS), LED36.3 (VSS), LED37.3 (VSS), LED38.3 (VSS), LED39.3 (VSS), LED4.3 (VSS), LED40.3 (VSS), LED41.3 (VSS), LED42.3 (VSS), LED43.3 (VSS), LED44.3 (VSS), LED45.3 (VSS), LED46.3 (VSS), LED47.3 (VSS), LED48.3 (VSS), LED49.3 (VSS), LED5.3 (VSS), LED50.3 (VSS), LED51.3 (VSS), LED52.3 (VSS), LED53.3 (VSS), LED54.3 (VSS), LED55.3 (VSS), LED56.3 (VSS), LED57.3 (VSS), LED58.3 (VSS), LED59.3 (VSS), LED6.3 (VSS), LED60.3 (VSS), LED61.3 (VSS), LED62.3 (VSS), LED63.3 (VSS), LED64.3 (VSS), LED65.3 (VSS), LED66.3 (VSS), LED67.3 (VSS), LED68.3 (VSS), LED69.3 (VSS), LED7.3 (VSS), LED70.3 (VSS), LED71.3 (VSS), LED72.3 (VSS), LED73.3 (VSS), LED74.3 (VSS), LED75.3 (VSS), LED76.3 (VSS), LED8.3 (VSS), LED9.3 (VSS), U2.GND
- net VCC: now reaches OL1.2 (VCC)
- net VCC: now also J1.1 (VCC), LED1.1 (VDD), LED10.1 (VDD), LED11.1 (VDD), LED12.1 (VDD), LED13.1 (VDD), LED14.1 (VDD), LED15.1 (VDD), LED16.1 (VDD), LED17.1 (VDD), LED18.1 (VDD), LED19.1 (VDD), LED2.1 (VDD), LED20.1 (VDD), LED21.1 (VDD), LED22.1 (VDD), LED23.1 (VDD), LED24.1 (VDD), LED25.1 (VDD), LED26.1 (VDD), LED27.1 (VDD), LED28.1 (VDD), LED29.1 (VDD), LED3.1 (VDD), LED30.1 (VDD), LED31.1 (VDD), LED32.1 (VDD), LED33.1 (VDD), LED34.1 (VDD), LED35.1 (VDD), LED36.1 (VDD), LED37.1 (VDD), LED38.1 (VDD), LED39.1 (VDD), LED4.1 (VDD), LED40.1 (VDD), LED41.1 (VDD), LED42.1 (VDD), LED43.1 (VDD), LED44.1 (VDD), LED45.1 (VDD), LED46.1 (VDD), LED47.1 (VDD), LED48.1 (VDD), LED49.1 (VDD), LED5.1 (VDD), LED50.1 (VDD), LED51.1 (VDD), LED52.1 (VDD), LED53.1 (VDD), LED54.1 (VDD), LED55.1 (VDD), LED56.1 (VDD), LED57.1 (VDD), LED58.1 (VDD), LED59.1 (VDD), LED6.1 (VDD), LED60.1 (VDD), LED61.1 (VDD), LED62.1 (VDD), LED63.1 (VDD), LED64.1 (VDD), LED65.1 (VDD), LED66.1 (VDD), LED67.1 (VDD), LED68.1 (VDD), LED69.1 (VDD), LED7.1 (VDD), LED70.1 (VDD), LED71.1 (VDD), LED72.1 (VDD), LED73.1 (VDD), LED74.1 (VDD), LED75.1 (VDD), LED76.1 (VDD), LED8.1 (VDD), LED9.1 (VDD), U2.5V (+5V)
- net Col10: now reaches OL1.3 (SCL)
- net Col10: now also SW17.2, SW32.2, SW47.2, SW61.2, SW71.2, U2.3 (3(PWM)/SCL)
- net Col11: now reaches OL1.4 (SDA)
- net Col11: now also SW18.2, SW33.2, SW48.2, SW62.2, SW72.2, U2.2 (2/SDA)
- net en2: now reaches SW77.A
- net en2: now also U2.MO (MOSI)
- net en1: now reaches SW77.B
- net en1: now also U2.SS (RX_LED/SS)
- net at SW77.S1: now also D77.2 (A)
- net Row1: now reaches SW77.S2
- net Row1: now also D1.1 (K), D2.1 (K), D3.1 (K), D4.1 (K), D5.1 (K), D6.1 (K), D7.1 (K), U2.A4
- net LED: now reaches J1.2 (LED)
- net LED: now also LED1.4 (DIN), U2.TX (1/TX)
- new net: D36.2 (A), SW36.1
- new net: LED30.2 (DOUT), LED31.4 (DIN)
- new net: LED29.2 (DOUT), LED30.4 (DIN)
- new net: LED1.2 (DOUT), LED2.4 (DIN)
- new net: D49.2 (A), SW49.1
- new net: D2.2 (A), SW2.1
- new net: LED31.2 (DOUT), LED32.4 (DIN)
- new net: D9.2 (A), SW9.1
- new net: LED46.2 (DOUT), LED47.4 (DIN)
- new net: LED45.2 (DOUT), LED46.4 (DIN)
- new net: D15.2 (A), SW15.1
- new net: D42.2 (A), SW42.1
- new net: LED75.2 (DOUT), LED76.4 (DIN)
- new net: LED74.2 (DOUT), LED75.4 (DIN)
- new net: LED49.2 (DOUT), LED50.4 (DIN)
- new net: LED48.2 (DOUT), LED49.4 (DIN)
- new net: LED18.2 (DOUT), LED19.4 (DIN)
- new net: LED17.2 (DOUT), LED18.4 (DIN)
- new net: LED22.2 (DOUT), LED23.4 (DIN)
- new net: LED21.2 (DOUT), LED22.4 (DIN)
- new net: LED2.2 (DOUT), LED3.4 (DIN)
- new net: LED33.2 (DOUT), LED34.4 (DIN)
- new net: LED32.2 (DOUT), LED33.4 (DIN)
- new net: D69.2 (A), SW69.1
- new net: D60.2 (A), SW60.1
- new net: D12.2 (A), SW12.1
- new net: LED58.2 (DOUT), LED59.4 (DIN)
- new net: LED57.2 (DOUT), LED58.4 (DIN)
- new net: LED16.2 (DOUT), LED17.4 (DIN)
- new net: D37.2 (A), SW37.1
- new net: LED28.2 (DOUT), LED29.4 (DIN)
- new net: D62.2 (A), SW62.1
- new net: D57.2 (A), SW57.1
- new net: LED70.2 (DOUT), LED71.4 (DIN)
- new net: LED69.2 (DOUT), LED70.4 (DIN)
- new net: LED50.2 (DOUT), LED51.4 (DIN)
- new net: D17.2 (A), SW17.1
- new net: D53.2 (A), SW53.1
- new net: D23.2 (A), SW23.1
- new net: D31.2 (A), SW31.1
- new net: D43.2 (A), SW43.1
- new net: D26.2 (A), SW26.1
- new net: LED52.2 (DOUT), LED53.4 (DIN)
- new net: LED51.2 (DOUT), LED52.4 (DIN)
- new net: LED23.2 (DOUT), LED24.4 (DIN)
- new net: LED63.2 (DOUT), LED64.4 (DIN)
- new net: LED62.2 (DOUT), LED63.4 (DIN)
- new net: LED20.2 (DOUT), LED21.4 (DIN)
- new net: D50.2 (A), SW50.1
- new net: D19.2 (A), SW19.1
- new net: D16.2 (A), SW16.1
- new net: D41.2 (A), SW41.1
- new net: D3.2 (A), SW3.1
- new net: D55.2 (A), SW55.1
- new net: LED26.2 (DOUT), LED27.4 (DIN)
- new net: LED25.2 (DOUT), LED26.4 (DIN)
- new net: D47.2 (A), SW47.1
- new net: LED72.2 (DOUT), LED73.4 (DIN)
- new net: LED71.2 (DOUT), LED72.4 (DIN)
- new net: D4.2 (A), SW4.1
- new net: D71.2 (A), SW71.1
- new net: D38.2 (A), SW38.1
- new net: D5.2 (A), SW5.1
- new net: LED8.2 (DOUT), LED9.4 (DIN)
- new net: LED7.2 (DOUT), LED8.4 (DIN)
- new net: D32.2 (A), SW32.1
- new net: LED19.2 (DOUT), LED20.4 (DIN)
- new net: D51.2 (A), SW51.1
- new net: D48.2 (A), SW48.1
- new net: D75.2 (A), SW75.1
- new net: D20.2 (A), SW20.1
- new net: D74.2 (A), SW74.1
- new net: LED38.2 (DOUT), LED39.4 (DIN)
- new net: LED37.2 (DOUT), LED38.4 (DIN)
- new net: D68.2 (A), SW68.1
- new net: D64.2 (A), SW64.1
- new net: D73.2 (A), SW73.1
- new net: D22.2 (A), SW22.1
- new net: D58.2 (A), SW58.1
- new net: D28.2 (A), SW28.1
- new net: D10.2 (A), SW10.1
- new net: LED68.2 (DOUT), LED69.4 (DIN)
- new net: LED67.2 (DOUT), LED68.4 (DIN)
- new net: D45.2 (A), SW45.1
- new net: D6.2 (A), SW6.1
- new net: D29.2 (A), SW29.1
- new net: D21.2 (A), SW21.1
- new net: D18.2 (A), SW18.1
- new net: D59.2 (A), SW59.1
- new net: D76.2 (A), SW76.1
- new net: D11.2 (A), SW11.1
- new net: D27.2 (A), SW27.1
- new net: D61.2 (A), SW61.1
- new net: D65.2 (A), SW65.1
- new net: D40.2 (A), SW40.1
- new net: LED27.2 (DOUT), LED28.4 (DIN)
- new net: LED36.2 (DOUT), LED37.4 (DIN)
- new net: D63.2 (A), SW63.1
- new net: LED35.2 (DOUT), LED36.4 (DIN)
- new net: LED34.2 (DOUT), LED35.4 (DIN)
- new net: D25.2 (A), SW25.1
- new net: D72.2 (A), SW72.1
- new net: D30.2 (A), SW30.1
- new net: D34.2 (A), SW34.1
- new net: LED73.2 (DOUT), LED74.4 (DIN)
- new net: LED6.2 (DOUT), LED7.4 (DIN)
- new net: LED65.2 (DOUT), LED66.4 (DIN)
- new net: LED64.2 (DOUT), LED65.4 (DIN)
- new net: LED43.2 (DOUT), LED44.4 (DIN)
- new net: LED42.2 (DOUT), LED43.4 (DIN)
- new net: D24.2 (A), SW24.1
- new net: D35.2 (A), SW35.1
- new net: D13.2 (A), SW13.1
- new net: D56.2 (A), SW56.1
- new net: D70.2 (A), SW70.1
- new net: D33.2 (A), SW33.1
- new net: D8.2 (A), SW8.1
- new net: D1.2 (A), SW1.1
- new net: LED66.2 (DOUT), LED67.4 (DIN)
- new net: D54.2 (A), SW54.1
- new net: LED3.2 (DOUT), LED4.4 (DIN)
- new net: LED5.2 (DOUT), LED6.4 (DIN)
- new net: LED4.2 (DOUT), LED5.4 (DIN)
- new net: D67.2 (A), SW67.1
- new net: D39.2 (A), SW39.1
- new net: D52.2 (A), SW52.1
- new net: LED53.2 (DOUT), LED54.4 (DIN)
- new net: LED14.2 (DOUT), LED15.4 (DIN)
- new net: LED13.2 (DOUT), LED14.4 (DIN)
- new net: LED54.2 (DOUT), LED55.4 (DIN)
- new net: D14.2 (A), SW14.1
- new net: LED61.2 (DOUT), LED62.4 (DIN)
- new net: D46.2 (A), SW46.1
- new net: D66.2 (A), SW66.1
- new net: LED55.2 (DOUT), LED56.4 (DIN)
- new net: LED60.2 (DOUT), LED61.4 (DIN)
- new net: LED56.2 (DOUT), LED57.4 (DIN)
- new net: LED39.2 (DOUT), LED40.4 (DIN)
- new net: LED12.2 (DOUT), LED13.4 (DIN)
- new net: LED44.2 (DOUT), LED45.4 (DIN)
- new net: D44.2 (A), SW44.1
- new net: LED59.2 (DOUT), LED60.4 (DIN)
- new net: LED10.4 (DIN), LED9.2 (DOUT)
- new net: LED47.2 (DOUT), LED48.4 (DIN)
- new net: LED24.2 (DOUT), LED25.4 (DIN)
- new net: LED11.2 (DOUT), LED12.4 (DIN)
- new net: LED10.2 (DOUT), LED11.4 (DIN)
- new net: D7.2 (A), SW7.1
- new net: LED15.2 (DOUT), LED16.4 (DIN)
- new net: LED41.2 (DOUT), LED42.4 (DIN)
- new net: LED40.2 (DOUT), LED41.4 (DIN)
- new net Col1: SW1.2, SW23.2, SW38.2, SW52.2, SW67.2, SW8.2, U2.12 (12/A11)
- new net Col12: SW19.2, SW34.2, SW49.2, SW63.2, SW73.2, U2.A5
- new net Col13: SW20.2, SW35.2, SW50.2, SW64.2, SW74.2, U2.MI (MISO)
- new net Col14: SW21.2, SW36.2, SW65.2, SW75.2, U2.SCK
- new net Col15: D77.1 (K), SW22.2, SW37.2, SW51.2, SW66.2, SW76.2, U2.RX (0/RX)
- new net Col2: SW24.2, SW39.2, SW53.2, SW68.2, SW9.2, U2.11 (11(PWM))
- new net Col3: SW10.2, SW2.2, SW25.2, SW40.2, SW54.2, SW69.2, U2.10 (10(PWM)/A10)
- new net Col4: SW11.2, SW26.2, SW3.2, SW41.2, SW55.2, U2.9 (9(PWM)/A9)
- new net Col5: SW12.2, SW27.2, SW4.2, SW42.2, SW56.2, U2.8 (8/A8)
- new net Col6: SW13.2, SW28.2, SW43.2, SW5.2, SW57.2, U2.7
- new net Col7: SW14.2, SW29.2, SW44.2, SW58.2, SW6.2, SW70.2, U2.6 (6(PWM)/A7)
- new net Col8: SW16.2, SW31.2, SW46.2, SW60.2, U2.4 (4/A6)
- new net Col9: SW15.2, SW30.2, SW45.2, SW59.2, SW7.2, U2.5 (5(PWM))
- new net Row2: D10.1 (K), D11.1 (K), D12.1 (K), D13.1 (K), D14.1 (K), D15.1 (K), D16.1 (K), D17.1 (K), D18.1 (K), D19.1 (K), D20.1 (K), D21.1 (K), D22.1 (K), D8.1 (K), D9.1 (K), U2.A3
- new net Row3: D23.1 (K), D24.1 (K), D25.1 (K), D26.1 (K), D27.1 (K), D28.1 (K), D29.1 (K), D30.1 (K), D31.1 (K), D32.1 (K), D33.1 (K), D34.1 (K), D35.1 (K), D36.1 (K), D37.1 (K), U2.13 (13(PWM))
- new net Row4: D38.1 (K), D39.1 (K), D40.1 (K), D41.1 (K), D42.1 (K), D43.1 (K), D44.1 (K), D45.1 (K), D46.1 (K), D47.1 (K), D48.1 (K), D49.1 (K), D50.1 (K), D51.1 (K), U2.A0
- new net Row5: D52.1 (K), D53.1 (K), D54.1 (K), D55.1 (K), D56.1 (K), D57.1 (K), D58.1 (K), D59.1 (K), D60.1 (K), D61.1 (K), D62.1 (K), D63.1 (K), D64.1 (K), D65.1 (K), D66.1 (K), U2.A1
- new net Row6: D67.1 (K), D68.1 (K), D69.1 (K), D70.1 (K), D71.1 (K), D72.1 (K), D73.1 (K), D74.1 (K), D75.1 (K), D76.1 (K), U2.A2
- no-connect marks 0 -> 5
Other:
- moved on the sheet: J1, OL1, SW77
